Commit message: update up-to-date urdf file of zackon

File: src/view_robot/urdf/robot_description.urdf (robot description, URDF)
Before this commit: robot view_robot_pkg, 8 links, 7 joints
Links:
- removed link lidar_link
- added link front_lidar_link, mass 0.0350818392125044; collision mesh filename=package://view_robot_pkg/meshes/front_lidar_link.STL; visual mesh filename=package://view_robot_pkg/meshes/front_lidar_link.STL
- added link rear_lidar_link, mass 0.0350818392110918; collision mesh filename=package://view_robot_pkg/meshes/rear_lidar_link.STL; visual mesh filename=package://view_robot_pkg/meshes/rear_lidar_link.STL
- link base_link: mass 10.432 -> 12.2572549705629
- link left_casterwheel_after_Link: mass 0.050885 -> 0.0508845884047379
- link left_casterwheel_before_Link: mass 0.050885 -> 0.0508845884047379
- link leftwheel_Link: mass 0.19451 -> 0.194507281551966
- link right_casterwheel_after_Link: mass 0.050885 -> 0.0508845884047379
- link right_casterwheel_before_Link: mass 0.050885 -> 0.0508845884047379
Joints:
- removed joint lidar_joint
- added joint front_lidar_joint: type fixed, parent base_link, child front_lidar_link, origin xyz=0.26014 0 0.18998 rpy=0 0 3.1416, axis 0 0 0
- added joint rear_lidar_joint: type fixed, parent base_link, child rear_lidar_link, origin xyz=-0.260140349955004 0 0.189977482585341 rpy=0 0 0, axis 0 0 0
- joint left_casterwheel_after_joint: origin xyz=-0.18642 -0.15554 0.062462 rpy=1.5708 0 0 -> xyz=-0.223 0.15515 0.02943 rpy=-1.5708 0 0
- joint left_casterwheel_before_joint: origin xyz=0.25358 -0.15543 0.062462 rpy=1.5708 0 0 -> xyz=0.217 0.15504 0.02943 rpy=-1.5708 0 0
- joint leftwheel_joint: origin xyz=0.03658 -0.14538 0.06286 rpy=1.5708 0 0 -> xyz=0 0.14499 0.028031 rpy=-1.5708 0 0
- joint right_casterwheel_after_joint: origin xyz=-0.18642 0.15447 0.062462 rpy=1.5708 0 0 -> xyz=-0.223 -0.15486 0.02943 rpy=-1.5708 0 0
- joint right_casterwheel_before_joint: origin xyz=0.25359 0.15433 0.062462 rpy=1.5708 0 0 -> xyz=0.217 -0.15486 0.02943 rpy=-1.5708 0 0
- joint rightwheel_joint: origin xyz=0.03658 0.14462 0.06286 rpy=1.5708 0 0 -> xyz=0 -0.14501 0.028031 rpy=-1.5708 0 0
